File: mainboard.kicad_sch (KiCad schematic)
At the start: 42 parts, among them J1 Micro_SD_Card, U1 RK3568, U2 RK809-1, Y1 24MHz, Y2 32.7kHz

Commit message: did a little bit more work on the microsd card, still incomplete, just pushing so other people can work on this
Parts:
- removed J1: Micro_SD_Card, symbol Connector:Micro_SD_Card
- added C36: 100nF X5R 10V, symbol Device:C_Small
- added D1: ESD9B3.3ST5G, Diode_SMD:D_SOD-923, symbol Diode:ESD9B3.3ST5G
- added J1: Micro_SD_Card_Det1, symbol Connector:Micro_SD_Card_Det1
- added R3: 22ohm 5%, symbol Device:R_Small
Connections:
- net GND: now also C36.2, J1.10 (SHIELD), J1.6 (VSS)
- net SDMMC0_D2/ARMJTAG_TCK: now reaches U1.H26 (GPIO1_D7_U)
- net SDMMC0_CMD: now reaches U1.H27 (GPIO2_A1_U)
- net at U1.H28 (GPIO2_A2_D): now also R3.2
- net SDMMC0_D3/ARMJTAG_TMS: now reaches U1.J23 (GPIO2_A0_U)
- net SDMMC0_D1: now reaches U1.J24 (GPIO1_D6_U)
- net SDMMC0_D0: now reaches U1.J25 (GPIO1_D5_U)
- net VCCIO_SD: now reaches U1.L22 (VCCIO3)
- net VCCIO_SD: now also C36.1
- net SDMMC0_DET: now reaches U1.Y22 (GPIO0_A4_U)
- new net SDMMC0_CLK: R3.1
